File: schematic/platform/platform.sch (KiCad schematic (older format))
At the start: 4 parts, among them J1 PLATFORM_CONNECTOR, J2 KY-018 PHOTORESISTOR MODULE, U1 HC-SR04

Commit message: Update schematic with the zakhar_kicadlib submodule
Parts:
- removed J1: PLATFORM_CONNECTOR, symbol Connector:Conn_01x08_Female
- removed J2: KY-018 PHOTORESISTOR MODULE, symbol Connector:Conn_01x03_Male
- removed U1: HC-SR04, XCVR_HC-SR04, symbol HC-SR04:HC-SR04
- added BT1: PowerBank_2xOUT, symbol zk_modules:PowerBank_2xOUT
- added J1: Conn_ZKP_1.3, symbol zk_connectors:Conn_ZKP_1.3
- added SW1: SW_SPDT, symbol Switch:SW_SPDT
- added U1: KY-018, symbol zk_modules:KY-018
- added U2: HC-SR04, XCVR_HC-SR04, symbol zk_modules:HC-SR04
Connections:
- wire segments 21 -> 25
Other:
- note removed: "+3V OUT"
- note removed: "+5V IN"
- note removed: "+5V OUT"
- note removed: "GND"
- note removed: "RESET"
- note removed: "SCK"
- note removed: "SDA"
- note removed: "SIGNAL"
- note removed: "VCC"
- moved on the sheet: A1
